Commit message: modified:   ros_arm/arm/urdf/arm_1_gazebo.urdf 	deleted:    ros_arm/arm/urdf/test.urdf 	modified:   ros_arm/arm/xacro/arm_1.xacro 	new file:   ros_arm/config/controllers/arm_1_gazebo_control.yaml 	renamed:    ros_arm/config/arm_1.rviz -> ros_arm/config/rviz/arm_1.rviz 	modified:   ros_arm/launch/arm_1_gazebo.launch 	new file:   ros_arm/launch/arm_1_gazebo_control.launch 	modified:   ros_arm/launch/arm_1_rviz.launch 	modified:   Moveit/moveit_resources (untracked content) 	modified:   Moveit/panda_moveit_config (modified content)

File: ros_arm/arm/urdf/arm_1_gazebo.urdf (robot description, URDF)
Before this commit: robot mycar, 1 links, 0 joints
Links:
- added link bottom_link; collision box size=1 1 0.02; visual box size=1 1 0.02
- added link grasping_frame
- added link gripper_finger_link1; visual box size=${left_gripper_len} ${left_gripper_width} ${left_gripper_he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
- added link gripper_finger_link2; visual box size=${right_gripper_len} ${right_gripper_width} ${right_gripper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
- added link link1; collision cylinder length=${link1_len} radius=${link1_width}; visual cylinder length=${link1_len} radius=${link1_width}
- added link link2; collision cylinder length=${link2_len} radius=${link2_width}; visual cylinder length=${link2_len} radius=${link2_width}
- added link link3; collision cylinder length=${link3_len} radius=${link3_width}; visual cylinder length=${link3_len} radius=${link3_width}
- added link link4; collision cylinder length=${link4_len} radius=${link4_width}; visual cylinder length=${link4_len} radius=${link4_width}
- added link link5; collision cylinder length=${link5_len} radius=${link5_width}; visual cylinder length=${link5_len} radius=${link5_width}
- added link link6; collision cylinder length=${link6_len} radius=${link6_width}; visual cylinder length=${link6_len} radius=${link6_width}
- link base_link: mass 6 -> None; geometry collision box size=0.1 0.1 0.04; visual box size=0.1 0.1 0.04
Joints:
- added joint bottom_joint: type fixed, parent base_link, child bottom_link, origin xyz=0 0 0 rpy=0 0 0
- added joint finger_joint1: type prismatic, parent link6, child gripper_finger_link1, origin xyz=0.0 0 0, axis 0 1 0, limit lower=0 upper=0.06 effort=100 velocity=1.0
- added joint finger_joint2: type fixed, parent link6, child gripper_finger_link2, origin xyz=0.0 0 0
- added joint grasping_frame_joint: type fixed, parent link6, child grasping_frame, origin xyz=0.08 0 0 rpy=0 0 0
- added joint joint1: type revolute, parent base_link, child link1, origin xyz=0 0 0.02 rpy=0 ${M_PI/2} 0, axis -1 0 0, limit lower=-2.96 upper=2.96 effort=300 velocity=1
- added joint joint2: type revolute, parent link1, child link2, origin xyz=-${link1_len} 0 0.0 rpy=-${M_PI/2} 0 ${M_PI/2}, axis 1 0 0, limit lower=-2.35 upper=2.35 effort=300 velocity=1
- added joint joint3: type revolute, parent link2, child link3, origin xyz=0 0 ${link2_len} rpy=0 ${M_PI} 0, axis -1 0 0, limit lower=-2.62 upper=2.62 effort=300 velocity=1
- added joint joint4: type revolute, parent link3, child link4, origin xyz=0.0 0.0 -${link3_len} rpy=0 ${M_PI/2} ${M_PI}, axis 1 0 0, limit lower=-2.62 upper=2.62 effort=300 velocity=1
- added joint joint5: type revolute, parent link4, child link5, origin xyz=${link4_len} 0.0 0.0 rpy=0 ${M_PI/2} 0, axis 1 0 0, limit lower=-2.62 upper=2.62 effort=300 velocity=1
- added joint joint6: type revolute, parent link5, child link6, origin xyz=0 0 ${link4_len} rpy=${1.5*M_PI} -${M_PI/2} 0, axis 1 0 0, limit lower=-6.28 upper=6.28 effort=300 velocity=1

File: ros_arm/arm/xacro/arm_1.xacro (robot description, xacro)
@@ -1,7 +1,5 @@
-<?xml version="1.0" ?>
-<robot name="arm_1"
-    xmlns:xacro="http://wiki.ros.org/xacro">
-    <xacro:include filename="utils_inertia.xacro" />
-    <!-- /    COLOR    / -->
+<?xml version="1.0"?>
+<robot name="arm" xmlns:xacro="http://ros.org/wiki/xacro">
+    <!-- Defining the colors used in this robot -->
     <material name="Black">
         <color rgba="0 0 0 1"/>
@@ -16,219 +14,333 @@
         <color rgba="1 0 0 1"/>
     </material>
-    <!-- /    BASE    / -->
+    <!-- Constants -->
+    <xacro:property name="M_PI" value="3.14159"/>
+    <!-- link1 properties -->
+    <xacro:property name="link1_width" value="0.03" />
+    <xacro:property name="link1_len" value="0.10" />
+    <!-- link2 properties -->
+    <xacro:property name="link2_width" value="0.03" />
+    <xacro:property name="link2_len" value="0.14" />
+    <!-- link3 properties -->
+    <xacro:property name="link3_width" value="0.03" />
+    <xacro:property name="link3_len" value="0.22" />
+    <!-- link4 properties -->
+    <xacro:property name="link4_width" value="0.025" />
+    <xacro:property name="link4_len" value="0.06" />
+    <!-- link5 properties -->
+    <xacro:property name="link5_width" value="0.03" />
+    <xacro:property name="link5_len" value="0.06" />
+    <!-- link6 properties -->
+    <xacro:property name="link6_width" value="0.04" />
+    <xacro:property name="link6_len" value="0.02" />
+    <!-- Left gripper -->
+    <xacro:property name="left_gripper_len" value="0.08" />
+    <xacro:property name="left_gripper_width" value="0.01" />
+    <xacro:property name="left_gripper_height" value="0.01" />
+    <!-- Right gripper -->
+    <xacro:property name="right_gripper_len" value="0.08" />
+    <xacro:property name="right_gripper_width" value="0.01" />
+    <xacro:property name="right_gripper_height" value="0.01" />
+    <!-- Gripper frame -->
+    <xacro:property name="grasp_frame_radius" value="0.001" />
+    <!-- Inertial matrix -->
+    <xacro:macro name="inertial_matrix" params="mass">
+        <inertial>
+            <mass value="${mass}" />
+            <inertia ixx="1.0" ixy="0.0" ixz="0.0" iyy="0.5" iyz="0.0" izz="1.0" />
+        </inertial>
+    </xacro:macro>
+    <!-- ///////////////////////////////////////   bottom_joint   ////////////////////////////////////////// -->
+    <joint name="bottom_joint" type="fixed">
+        <origin xyz="0 0 0" rpy="0 0 0" />
+        <parent link="base_link"/>
+        <child link="bottom_link"/>
+    </joint>
+    <link name="bottom_link">
+        <visual>
+              <origin xyz=" 0 0 -0.02"  rpy="0 0 0"/>
+                  <geometry>
+                       <box size="0.1 0.1 0.02" />
+                  </geometry>
+              <material name="Brown" />
+        </visual>
+        <collision>
+            <origin xyz=" 0 0 -0.02"  rpy="0 0 0"/>
+            <geometry>
+                <box size="0.1 0.1 0.02" />
+            </geometry>
+        </collision>
+        <xacro:inertial_matrix mass="500"/>
+    </link>
+    <!-- /////////////////////////////////////   BASE LINK    ////////////////////////////////////////////// -->
     <link name="base_link">
         <visual>
-            <origin rpy="0 0 0" xyz="0 0 0"/>
-            <geometry>
-                <cylinder length="0.04" radius="0.05"/>
-            </geometry>
-            <material name="White"/>
-        </visual>
-        <collision>
-            <origin rpy="0 0 0" xyz="0 0 0"/>
-            <geometry>
-                <cylinder length="0.04" radius="0.05"/>
-            </geometry>
-        </collision>
-        <xacro:cylinder_inertial_matrix m = "0.1" r = "0.05" h = "0.04"/>
-    </link>
-    <!-- /   LINK1  // -->
-    <link name="link1">
-        <visual>
-            <origin rpy="0 1.5707 0" xyz="-0.05 0 0"/>
-            <geometry>
-                <cylinder length="0.1" radius="0.03"/>
-            </geometry>
-            <material name="Blue"/>
-        </visual>
-        <collision>
-            <origin rpy="0 1.5707 0" xyz="-0.05 0 0"/>
-            <geometry>
-                <cylinder length="0.1" radius="0.03"/>
-            </geometry>
-        </collision>
-        <xacro:cylinder_inertial_matrix m = "0.1" r = "0.03" h = "0.1"/>
+            <origin xyz="0 0 0" rpy="0 0 0" />
+            <geometry>
+                <box size="0.1 0.1 0.04" />
+            </geometry>
+            <material name="White" />
+        </visual>
+        <collision>
+            <origin xyz="0 0 0" rpy="0 0 0" />
+            <geometry>
+                <box size="0.1 0.1 0.04" />
+            </geometry>
+        </collision>
+        <xacro:inertial_matrix mass="1"/>
     </link>
     <joint name="joint1" type="revolute">
         <parent link="base_link"/>
         <child link="link1"/>
-        <origin rpy="0 1.5707 0" xyz="0 0 0.02"/>
-        <axis xyz="-1 0 0"/>
-        <limit effort="300" lower="-3.14159" upper="3.14159" velocity="1"/>
-    </joint>
-    <!-- ///   LINK2  // -->
-    <link name="link2">
-        <visual>
-            <origin rpy="0 0 0" xyz="0 0 0.07"/>
-            <geometry>
-                <cylinder length="0.14" radius="0.03"/>
-            </geometry>
-            <material name="White"/>
-        </visual>
-        <collision>
-            <origin rpy="0 0 0" xyz="0 0 0.07"/>
-            <geometry>
-                <cylinder length="0.14" radius="0.03"/>
-            </geometry>
-        </collision>
-        <xacro:cylinder_inertial_matrix m = "0.1" r = "0.03" h = "0.14"/>
+        <origin xyz="0 0 0.02" rpy="0 ${M_PI/2} 0" />
+        <axis xyz="-1 0 0" />
+        <limit effort="300" velocity="1" lower="-2.96" upper="2.96"/>
+        <dynamics damping="50" friction="1"/>
+    </joint>
+    <!-- /////////////////////////////////////   LINK1  ////////////////////////////////////////////// -->
+    <link name="link1" >
+        <visual>
+            <origin xyz="-${link1_len/2} 0 0" rpy="0 ${M_PI/2} 0" />
+            <geometry>
+                <cylinder radius="${link1_width}" length="${link1_len}"/>
+            </geometry>
+            <material name="Blue" />
+        </visual>
+        <collision>
+            <origin xyz="-${link1_len/2} 0 0" rpy="0 ${M_PI/2} 0" />
+            <geometry>
+                <cylinder radius="${link1_width}" length="${link1_len}"/>
+            </geometry>
+        </collision>
+        <xacro:inertial_matrix mass="1"/>
     </link>
     <joint name="joint2" type="revolute">
         <parent link="link1"/>
         <child link="link2"/>
-        <origin rpy="-1.5707 0 1.5707" xyz="-0.1 0 0.0"/>
-        <axis xyz="1 0 0"/>
-        <limit effort="300" lower="-3.14159" upper="3.14159" velocity="1"/>
-    </joint>
-    <!-- /   LINK3  / -->
-    <link name="link3">
-        <visual>
-            <origin rpy="0 0 0" xyz="0 0 -0.075"/>
-            <geometry>
-                <cylinder length="0.15" radius="0.03"/>
-            </geometry>
-            <material name="Blue"/>
-        </visual>
-        <collision>
-            <origin rpy="0 0 0" xyz="0 0 -0.075"/>
-            <geometry>
-                <cylinder length="0.15" radius="0.03"/>
-            </geometry>
-        </collision>
-        <xacro:cylinder_inertial_matrix m = "0.1" r = "0.03" h = "0.15"/>
+        <origin xyz="-${link1_len} 0 0.0" rpy="-${M_PI/2} 0 ${M_PI/2}" />
+        <axis xyz="1 0 0" />
+        <limit effort="300" velocity="1" lower="-2.35" upper="2.35" />
+        <dynamics damping="50" friction="1"/>
+    </joint>
+    <!-- ///////////////////////////////////////   LINK2  ////////////////////////////////////////////// -->
+    <link name="link2" >
+        <visual>
+            <origin xyz="0 0 ${link2_len/2}" rpy="0 0 0" />
+            <geometry>
+                <cylinder radius="${link2_width}" length="${link2_len}"/>
+            </geometry>
+            <material name="White" />
+        </visual>
+        <collision>
+            <origin xyz="0 0 ${link2_len/2}" rpy="0 0 0" />
+            <geometry>
+                <cylinder radius="${link2_width}" length="${link2_len}"/>
+            </geometry>
+        </collision>
+        <xacro:inertial_matrix mass="1"/>
     </link>
     <joint name="joint3" type="revolute">
         <parent link="link2"/>
         <child link="link3"/>
-        <origin rpy="0 3.14159 0" xyz="0 0 0.14"/>
-        <axis xyz="-1 0 0"/>
-        <limit effort="300" lower="-3.14159" upper="3.14159" velocity="1"/>
-    </joint>
-    <!-- ///   LINK4   -->
-    <link name="link4">
-        <visual>
-            <origin rpy="0 1.5707 0" xyz="0.03 0 0"/>
-            <geometry>
-                <cylinder length="0.06" radius="0.025"/>
-            </geometry>
-            <material name="Black"/>
-        </visual>
-        <collision>
-            <origin rpy="0 1.5707 0" xyz="0.03 0 0"/>
-            <geometry>
-                <cylinder length="0.06" radius="0.025"/>
-            </geometry>
-        </collision>
-        <xacro:cylinder_inertial_matrix m = "0.1" r = "0.025" h = "0.06"/>
+        <origin xyz="0 0 ${link2_len}" rpy="0 ${M_PI} 0" />
+        <axis xyz="-1 0 0" />
+        <limit effort="300" velocity="1" lower="-2.62" upper="2.62" />
+        <dynamics damping="50" friction="1"/>
+    </joint>
+    <!-- /////////////////////////////////   LINK3  ///////////////////////////////////////////////////// -->
+    <link name="link3" >
+        <visual>
+            <origin xyz="0 0 -${link3_len/2}" rpy="0 0 0" />
+            <geometry>
+                <cylinder radius="${link3_width}" length="${link3_len}"/>
+            </geometry>
+            <material name="Blue" />
+        </visual>
+        <collision>
+            <origin xyz="0 0 -${link3_len/2}" rpy="0 0 0" />
+            <geometry>
+                <cylinder radius="${link3_width}" length="${link3_len}"/>
+            </geometry>
+        </collision>
+        <xacro:inertial_matrix mass="1"/>
     </link>
     <joint name="joint4" type="revolute">
         <parent link="link3"/>
         <child link="link4"/>
-        <origin rpy="0 1.5707 3.14159" xyz="0.0 0.0 -0.15"/>
-        <axis xyz="1 0 0"/>
-        <limit effort="300" lower="-3.14159" upper="3.14159" velocity="1"/>
-    </joint>
-    <!-- //   LINK5  / -->
-    <link name="link5">
-        <visual>
-            <origin rpy="0 0 0" xyz="0 0 0.03"/>
-            <geometry>
-                <cylinder length="0.06" radius="0.03"/>
-            </geometry>
-            <material name="White"/>
-        </visual>
-        <collision>
-            <origin rpy="0 0 0" xyz="0 0 0.03"/>
-            <geometry>
-                <cylinder length="0.06" radius="0.03"/>
-            </geometry>
-        </collision>
-        <xacro:cylinder_inertial_matrix m = "0.1" r = "0.03" h = "0.06"/>
+        <origin xyz="0.0 0.0 -${link3_len}" rpy="0 ${M_PI/2} ${M_PI}" />
+        <axis xyz="1 0 0" />
+        <limit effort="300" velocity="1" lower="-2.62" upper="2.62" />
+        <dynamics damping="50" friction="1"/>
+    </joint>
+    <!-- ///////////////////////////////////   LINK4  //////////////////////////////////////////////// -->
+    <link name="link4" >
+        <visual>
+            <origin xyz="${link4_len/2} 0 0" rpy="0 ${M_PI/2} 0" />
+            <geometry>
+                <cylinder radius="${link4_width}" length="${link4_len}"/>
+            </geometry>
+            <material name="Black" />
+        </visual>
+        <collision>
+            <origin xyz="${link4_len/2} 0 0" rpy="0 ${M_PI/2} 0" />
+            <geometry>
+                <cylinder radius="${link4_width}" length="${link4_len}"/>
+            </geometry>
+        </collision>
+        <xacro:inertial_matrix mass="1"/>
     </link>
     <joint name="joint5" type="revolute">
         <parent link="link4"/>
         <child link="link5"/>
-        <origin rpy="0 1.5707 0" xyz="0.06 0.0 0.0"/>
-        <axis xyz="1 0 0"/>
-        <limit effort="300" lower="-3.14159" upper="3.14159" velocity="1"/>
-    </joint>
-    <!--    LINK6  / -->
-    <link name="link6">
-        <visual>
-            <origin rpy="0 1.5707 0" xyz="0.01 0 0 "/>
-            <geometry>
-                <cylinder length="0.02" radius="0.04"/>
-            </geometry>
-            <material name="Blue"/>
-        </visual>
-        <collision>
-            <origin rpy="0 1.5707 0" xyz="0.01 0 0 "/>
-            <geometry>
-                <cylinder length="0.02" radius="0.04"/>
-            </geometry>
-        </collision>
-        <xacro:cylinder_inertial_matrix m = "0.1" r = "0.04" h = "0.02"/>
+        <origin xyz="${link4_len} 0.0 0.0" rpy="0 ${M_PI/2} 0" />
+        <axis xyz="1 0 0" />
+        <limit effort="300" velocity="1" lower="-2.62" upper="2.62" />
+        <dynamics damping="50" friction="1"/>
+    </joint>
+    <!-- //////////////////////////////////   LINK5  ///////////////////////////////////////////////// -->
+    <link name="link5">
+        <visual>
+            <origin xyz="0 0 ${link4_len/2}" rpy="0 0 0" />
+            <geometry>
+                <cylinder radius="${link5_width}" length="${link5_len}"/>
+            </geometry>
+            <material name="White" />
+        </visual>
+        <collision>
+            <origin xyz="0 0 ${link4_len/2} " rpy="0 0 0" />
+            <geometry>
+                <cylinder radius="${link5_width}" length="${link5_len}"/>
+            </geometry>
+        </collision>
+        <xacro:inertial_matrix mass="1"/>
     </link>
     <joint name="joint6" type="revolute">
         <parent link="link5"/>
         <child link="link6"/>
-        <origin rpy="4.712385 -1.5707 0" xyz="0 0 0.06"/>
-        <axis xyz="1 0 0"/>
-        <limit effort="300" lower="-6.28318" upper="6.28318" velocity="1"/>
-    </joint>
-    <!-- //   GRIPPER   // -->
-    <link name="gripper_finger_link1">
-        <visual>
-            <origin rpy="0 1.5707 0" xyz="0.03 0 0"/>
-            <geometry>
-                <box size="0.03 0.01 0.06"/>
-            </geometry>
-            <material name="White"/>
-        </visual>
-        <collision>
-            <origin rpy="0 1.5707 0" xyz="0.03 0 0"/>
-            <geometry>
-                <box size="0.03 0.01 0.06"/>
-            </geometry>
-        </collision>
-        <xacro:Box_inertial_matrix m = "0.1" l = "0.06" w = "0.01" h = "0.03"/>
-    </link>
-    <link name="gripper_finger_link2">
-        <visual>
-            <origin rpy="0 1.5707 0" xyz="0.03 0 0"/>
-            <geometry>
-                <box size="0.03 0.01 0.06"/>
-            </geometry>
-            <material name="White"/>
-        </visual>
-        <collision>
-            <origin rpy="0 1.5707 0" xyz="0.03 0 0"/>
-            <geometry>
-                <box size="0.03 0.01 0.06"/>
-            </geometry>
-        </collision>
-        <xacro:Box_inertial_matrix m = "0.1" l = "0.06" w = "0.01" h = "0.03"/>
+        <origin xyz="0 0 ${link4_len}" rpy="${1.5*M_PI} -${M_PI/2} 0" />
+        <axis xyz="1 0 0" />
+        <limit effort="300" velocity="1" lower="-6.28" upper="6.28" />
+        <dynamics damping="50" friction="1"/>
+    </joint>
+    <!-- ////////////////////////////////   LINK6  ///////////////////////////////////////////////// -->
+    <link name="link6">
+        <visual>
+            <origin xyz="${link6_len/2} 0 0 " rpy="0 ${M_PI/2} 0" />
+            <geometry>
+                <cylinder radius="${link6_width}" length="${link6_len}"/>
+            </geometry>
+            <material name="Blue" />
+        </visual>
+        <collision>
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