Commit message: Changes to be committed: 	modified:   ros_arm/arm/xacro/camera.xacro 	modified:   ros_arm/config/gazebo_world/arm_test.world 	modified:   ros_arm/launch/arm_gazebo.launch
Changes not staged for commit:
	modified:   Moveit/moveit_resources (untracked content)
	modified:   Moveit/panda_moveit_config (modified content)

File: ros_arm/arm/xacro/camera.xacro (robot description, xacro)
@@ -8,5 +8,5 @@
     <xacro:property name="camera_width" value="0.045" /> <!-- width(y) -->
     <xacro:property name="camera_height" value="0.025" /> <!-- height(z) -->
-    <xacro:property name="camera_x" value="0.08" /> <!-- connection_pos x -->
+    <xacro:property name="camera_x" value="0.02" /> <!-- connection_pos x -->
     <xacro:property name="camera_y" value="0.0" /> <!-- connection_pos y -->
     <xacro:property name="camera_z" value="0.0" /> <!-- connection_pos z -->
