Commit message: 1. modified camera model 2. modified finger model 3. add finger control 4. record6.mp4: finger moving

File: ros_arm/arm/xacro/arm.xacro (robot description, xacro)
@@ -245,5 +245,5 @@
         <origin xyz="0.0 0 0" />
         <axis xyz="0 1 0" />
-        <limit effort="100" lower="0" upper="0.025" velocity="1.0"/>
+        <limit effort="100" lower="0" upper="0.015" velocity="0.05"/>
         <dynamics damping="50" friction="1"/>
     </joint>
@@ -265,5 +265,5 @@
         <origin xyz="0.0 0 0" />
         <axis xyz="0 -1 0" />
-        <limit effort="100" lower="0" upper="0.025" velocity="1.0"/>
+        <limit effort="100" lower="0" upper="0.015" velocity="0.05"/>
         <dynamics damping="50" friction="1"/>
     </joint>

File: ros_arm/arm/xacro/camera.xacro (robot description, xacro)
@@ -5,8 +5,8 @@
     <xacro:include filename="utils_inertia.xacro" />
     <!-- properties -->
-    <xacro:property name="camera_length" value="0.01" /> <!-- length(x) -->
-    <xacro:property name="camera_width" value="0.045" /> <!-- width(y) -->
-    <xacro:property name="camera_height" value="0.025" /> <!-- height(z) -->
-    <xacro:property name="camera_x" value="0.02" /> <!-- connection_pos x -->
+    <xacro:property name="camera_length" value="0.001" /> <!-- length(x) -->
+    <xacro:property name="camera_width" value="0.01" /> <!-- width(y) -->
+    <xacro:property name="camera_height" value="0.01" /> <!-- height(z) -->
+    <xacro:property name="camera_x" value="0.0205" /> <!-- connection_pos x -->
     <xacro:property name="camera_y" value="0.0" /> <!-- connection_pos y -->
     <xacro:property name="camera_z" value="0.0" /> <!-- connection_pos z -->
@@ -35,5 +35,5 @@
     </joint>
     <gazebo reference="camera">
-        <material>Gazebo/Blue</material>
+        <material>Gazebo/Black</material>
     </gazebo>
 </robot>

Commit message: 1. modified camera frequency from 30Hz to 60Hz 2. added 4 boxes in gazebo world to test the camera and CV 3. added image_process.py to process the image from camera 4. added initial_mover.py to move the arm to camera-test initial position

File: ros_arm/arm/xacro/arm.xacro (robot description, xacro)
@@ -53,5 +53,5 @@
     <!-- ///////////////////////////////////////   bottom_joint   ////////////////////////////////////////// -->
     <joint name="bottom_joint" type="fixed">
-        <origin xyz="0 0 0" rpy="0 0 0" />
+        <origin xyz="0 0 -0.025" rpy="0 0 0" />
         <parent link="base_link"/>
         <child link="bottom_link"/>
@@ -59,17 +59,17 @@
     <link name="bottom_link">
         <visual>
-              <origin xyz=" 0 0 -0.02"  rpy="0 0 0"/>
+              <origin xyz=" 0 0 0"  rpy="0 0 0"/>
                   <geometry>
-                       <box size="0.1 0.1 0.02" />
+                       <box size="0.1 0.1 0.01" />
                   </geometry>
-              <material name="Brown" />
-        </visual>
-        <collision>
-            <origin xyz=" 0 0 -0.02"  rpy="0 0 0"/>
-            <geometry>
-                <box size="0.1 0.1 0.02" />
-            </geometry>
-        </collision>
-        <xacro:inertial_matrix mass="50000"/>
+              <material name="Blue" />
+        </visual>
+        <collision>
+            <origin xyz=" 0 0 0"  rpy="0 0 0"/>
+            <geometry>
+                <box size="0.1 0.1 0.01" />
+            </geometry>
+        </collision>
+        <xacro:inertial_matrix mass="1000"/>
     </link>
     <!-- /////////////////////////////////////   BASE LINK    ////////////////////////////////////////////// -->
@@ -291,5 +291,5 @@
     <!-- /////////////////////////////////   Gazebo   ////////////////////////////////////// -->
     <gazebo reference="bottom_link">
-        <material>Gazebo/White</material>
+        <material>Gazebo/Black</material>
     </gazebo>
     <gazebo reference="base_link">

File: ros_arm/arm/xacro/camera_sensor.xacro (robot description, xacro)
@@ -4,7 +4,7 @@
     <!-- set type as camara -->
     <sensor type="camera" name="rgb_camera">
-      <update_rate>30.0</update_rate> <!-- frequence -->
+      <update_rate>60.0</update_rate> <!-- frequence -->
       <!-- properties of camera -->
-      <camera name="head">
+      <camera name="rgb_camera">
         <horizontal_fov>1.3962634</horizontal_fov>
         <image>
@@ -31,5 +31,5 @@
         <cameraInfoTopicName>camera_info</cameraInfoTopicName>
         <frameName>camera</frameName>
-        <hackBaseline>0.07</hackBaseline>
+        <hackBaseline>0.0</hackBaseline>
         <distortionK1>0.0</distortionK1>
         <distortionK2>0.0</distortionK2>

Commit message: 1. modified details of arm.xacro 2. modified arm_conrtol in arm_conrtol.py 3. speed up image_process in image_process.py 4. f**k the awful original image_process.py

File: ros_arm/arm/xacro/arm.xacro (robot description, xacro)
@@ -21,8 +21,8 @@
     <!-- link2 properties -->
     <xacro:property name="link2_width" value="0.03" />
-    <xacro:property name="link2_len" value="0.22" />
+    <xacro:property name="link2_len" value="0.2" />
     <!-- link3 properties -->
     <xacro:property name="link3_width" value="0.03" />
-    <xacro:property name="link3_len" value="0.14" />
+    <xacro:property name="link3_len" value="0.2" />
     <!-- link4 properties -->
     <xacro:property name="link4_width" value="0.025" />
@@ -94,5 +94,5 @@
         <child link="link1"/>
         <origin xyz="0 0 0.02" rpy="0 ${M_PI/2} 0" />
-        <axis xyz="-1 0 0" />
+        <axis xyz="1 0 0" />
         <limit effort="300" velocity="1" lower="-2.96" upper="2.96"/>
         <dynamics damping="50" friction="1"/>
@@ -110,5 +110,5 @@
             <origin xyz="-${link1_len/2} 0 0" rpy="0 ${M_PI/2} 0" />
             <geometry>
-                <cylinder radius="${link1_width}" length="${link1_len}"/>
+                <cylinder radius="${link1_width/10}" length="${link1_len/10}"/>
             </geometry>
         </collision>
@@ -135,5 +135,5 @@
             <origin xyz="0 0 ${link2_len/2}" rpy="0 0 0" />
             <geometry>
-                <cylinder radius="${link2_width}" length="${link2_len}"/>
+                <cylinder radius="${link2_width/10}" length="${link2_len/10}"/>
             </geometry>
         </collision>
@@ -160,5 +160,5 @@
             <origin xyz="0 0 -${link3_len/2}" rpy="0 0 0" />
             <geometry>
-                <cylinder radius="${link3_width}" length="${link3_len}"/>
+                <cylinder radius="${link3_width/10}" length="${link3_len/10}"/>
             </geometry>
         </collision>
@@ -194,5 +194,5 @@
         <child link="link5"/>
         <origin xyz="${link4_len} 0.0 0.0" rpy="0 ${M_PI/2} 0" />
-        <axis xyz="1 0 0" />
+        <axis xyz="-1 0 0" />
         <limit effort="300" velocity="1" lower="-2.62" upper="2.62" />
         <dynamics damping="50" friction="1"/>

Commit message: v1

File: ros_arm/arm/xacro/arm.xacro (robot description, xacro)
@@ -1,4 +1,5 @@
 <?xml version="1.0"?>
-<robot name="arm" xmlns:xacro="http://ros.org/wiki/xacro">
+<robot name="arm"
+    xmlns:xacro="http://ros.org/wiki/xacro">
     <!-- Defining the colors used in this robot -->
     <material name="Black">
@@ -37,9 +38,9 @@
     <xacro:property name="left_gripper_len" value="0.08" />
     <xacro:property name="left_gripper_width" value="0.01" />
-    <xacro:property name="left_gripper_height" value="0.01" />
+    <xacro:property name="left_gripper_height" value="0.03" />
     <!-- Right gripper -->
     <xacro:property name="right_gripper_len" value="0.08" />
     <xacro:property name="right_gripper_width" value="0.01" />
-    <xacro:property name="right_gripper_height" value="0.01" />
+    <xacro:property name="right_gripper_height" value="0.03" />
     <!-- Gripper frame -->
     <xacro:property name="grasp_frame_radius" value="0.001" />
@@ -59,12 +60,12 @@
     <link name="bottom_link">
         <visual>
-              <origin xyz=" 0 0 0"  rpy="0 0 0"/>
-                  <geometry>
-                       <box size="0.1 0.1 0.01" />
-                  </geometry>
-              <material name="Blue" />
-        </visual>
-        <collision>
-            <origin xyz=" 0 0 0"  rpy="0 0 0"/>
+            <origin xyz=" 0 0 0" rpy="0 0 0"/>
+            <geometry>
+                <box size="0.1 0.1 0.01" />
+            </geometry>
+            <material name="Blue" />
+        </visual>
+        <collision>
+            <origin xyz=" 0 0 0" rpy="0 0 0"/>
             <geometry>
                 <box size="0.1 0.1 0.01" />
@@ -99,5 +100,5 @@
     </joint>
     <!-- /////////////////////////////////////   LINK1  ////////////////////////////////////////////// -->
-    <link name="link1" >
+    <link name="link1">
         <visual>
             <origin xyz="-${link1_len/2} 0 0" rpy="0 ${M_PI/2} 0" />
@@ -124,5 +125,5 @@
     </joint>
     <!-- ///////////////////////////////////////   LINK2  ////////////////////////////////////////////// -->
-    <link name="link2" >
+    <link name="link2">
         <visual>
             <origin xyz="0 0 ${link2_len/2}" rpy="0 0 0" />
@@ -149,5 +150,5 @@
     </joint>
     <!-- /////////////////////////////////   LINK3  ///////////////////////////////////////////////////// -->
-    <link name="link3" >
+    <link name="link3">
         <visual>
             <origin xyz="0 0 -${link3_len/2}" rpy="0 0 0" />
@@ -174,5 +175,5 @@
     </joint>
     <!-- ///////////////////////////////////   LINK4  //////////////////////////////////////////////// -->
-    <link name="link4" >
+    <link name="link4">
         <visual>
             <origin xyz="${link4_len/2} 0 0" rpy="0 ${M_PI/2} 0" />
@@ -258,4 +259,11 @@
             <material name="White" />
         </visual>
+        <collision>
+            <origin xyz="0.04 -0.03 0"/>
+            <geometry>
+                <box size="${left_gripper_len/2} ${left_gripper_width} ${left_gripper_height}" />
+            </geometry>
+        </collision>
+        <contact_coefficients mu="200.0" kp="0.0" kd="0.0"/>
         <xacro:inertial_matrix mass="1"/>
     </link>
@@ -277,4 +285,11 @@
             <material name="White" />
         </visual>
+        <collision>
+            <origin xyz="0.04 0.03 0"/>
+            <geometry>
+                <box size="${right_gripper_len/2} ${right_gripper_width} ${right_gripper_height}" />
+            </geometry>
+        </collision>
+        <contact_coefficients mu="200.0" kp="0.0" kd="0.0"/>
         <xacro:inertial_matrix mass="1"/>
     </link>
@@ -282,7 +297,7 @@
     <link name="grasping_frame"/>
     <joint name="grasping_frame_joint" type="fixed">
-      <parent link="link6"/>
-      <child link="grasping_frame"/>
-      <origin xyz="0.08 0 0" rpy="0 0 0"/>
+        <parent link="link6"/>
+        <child link="grasping_frame"/>
+        <origin xyz="0.08 0 0" rpy="0 0 0"/>
     </joint>
     <!-- /////////////////////////////////   camera   ////////////////////////////////////// -->
@@ -346,4 +361,19 @@
             <robotNamespace>/arm</robotNamespace>
         </plugin>
+        <plugin name="gazebo_grasp_fix" filename="libgazebo_grasp_fix.so">
+            <arm>
+                <arm_name>arm</arm_name>
+                <!-- <palm_link> hand_link_name  </palm_link> -->
+                <gripper_link> gripper_finger_link1 </gripper_link>
+                <gripper_link> gripper_finger_link2 </gripper_link>
+            </arm>
+            <forces_angle_tolerance>100</forces_angle_tolerance>
+            <update_rate>4</update_rate>
+            <grip_count_threshold>4</grip_count_threshold>
+            <max_grip_count>8</max_grip_count>
+            <release_tolerance>0.005</release_tolerance>
+            <disable_collisions_on_attach>false</disable_collisions_on_attach>
+            <contact_topic>__default_topic__</contact_topic>
+        </plugin>
     </gazebo>
 </robot>

Commit message: gripper fix test

File: ros_arm/arm/xacro/arm.xacro (robot description, xacro)
@@ -282,7 +282,13 @@
     <link name="grasping_frame"/>
     <joint name="grasping_frame_joint" type="fixed">
+<<<<<<< Updated upstream
       <parent link="link6"/>
       <child link="grasping_frame"/>
       <origin xyz="0.08 0 0" rpy="0 0 0"/>
+=======
+        <parent link="link6"/>
+        <child link="grasping_frame"/>
+        <origin xyz="0.08 0 0" rpy="0 0 .02"/>
+>>>>>>> Stashed changes
     </joint>
     <!-- /////////////////////////////////   camera   ////////////////////////////////////// -->
@@ -316,7 +322,35 @@
     <gazebo reference="gripper_finger_link1">
         <material>Gazebo/White</material>
+        <mu1>1000</mu1>
+        <mu2>1000</mu2>
+        <kp>1000000.0</kp>
+        <kd>100000.0</kd>
+        <slip1>0</slip1>
+        <slip2>0</slip2>
+        <minDepth>0.003</minDepth>
+        <maxVel>0</maxVel>
+        <torsional>
+            <ode>
+                <coefficient>1000000</coefficient>
+                <slip>0</slip>
+            </ode>
+        </torsional>
     </gazebo>
     <gazebo reference="gripper_finger_link2">
         <material>Gazebo/White</material>
+        <mu1>1000</mu1>
+        <mu2>1000</mu2>
+        <kp>1000000.0</kp>
+        <kd>100000.0</kd>
+        <slip1>0</slip1>
+        <slip2>0</slip2>
+        <minDepth>0.003</minDepth>
+        <maxVel>0</maxVel>
+        <torsional>
+            <ode>
+                <coefficient>1000000</coefficient>
+                <slip>0</slip>
+            </ode>
+        </torsional>
     </gazebo>
     <!-- Transmissions for ROS Control -->
@@ -346,4 +380,22 @@
             <robotNamespace>/arm</robotNamespace>
         </plugin>
+<<<<<<< Updated upstream
+=======
+        <plugin name="gazebo_grasp_fix" filename="libgazebo_grasp_fix.so">
+            <arm>
+                <arm_name>arm</arm_name>
+                <palm_link> link6 </palm_link>
+                <gripper_link> gripper_finger_link1 </gripper_link>
+                <gripper_link> gripper_finger_link2 </gripper_link>
+            </arm>
+            <forces_angle_tolerance>120</forces_angle_tolerance>
+            <update_rate>4</update_rate>
+            <grip_count_threshold>4</grip_count_threshold>
+            <max_grip_count>8</max_grip_count>
+            <release_tolerance>0.005</release_tolerance>
+            <disable_collisions_on_attach>false</disable_collisions_on_attach>
+            <contact_topic>__default_topic__</contact_topic>
+        </plugin>
+>>>>>>> Stashed changes
     </gazebo>
 </robot>

Commit message: fixed grasp of gripper

File: ros_arm/arm/xacro/arm.xacro (robot description, xacro)
@@ -36,11 +36,11 @@
     <xacro:property name="link6_len" value="0.02" />
     <!-- Left gripper -->
-    <xacro:property name="left_gripper_len" value="0.08" />
+    <xacro:property name="left_gripper_len" value="0.06" />
     <xacro:property name="left_gripper_width" value="0.01" />
-    <xacro:property name="left_gripper_height" value="0.03" />
+    <xacro:property name="left_gripper_height" value="0.01" />
     <!-- Right gripper -->
-    <xacro:property name="right_gripper_len" value="0.08" />
+    <xacro:property name="right_gripper_len" value="0.06" />
     <xacro:property name="right_gripper_width" value="0.01" />
-    <xacro:property name="right_gripper_height" value="0.03" />
+    <xacro:property name="right_gripper_height" value="0.01" />
     <!-- Gripper frame -->
     <xacro:property name="grasp_frame_radius" value="0.001" />
@@ -253,5 +253,5 @@
     <link name="gripper_finger_link1">
         <visual>
-            <origin xyz="0.04 -0.03 0"/>
+            <origin xyz="${link6_len+left_gripper_len/2} -0.03 0"/>
             <geometry>
                 <box size="${left_gripper_len} ${left_gripper_width} ${left_gripper_height}" />
@@ -260,10 +260,10 @@
         </visual>
         <collision>
-            <origin xyz="0.04 -0.03 0"/>
-            <geometry>
-                <box size="${left_gripper_len/2} ${left_gripper_width} ${left_gripper_height}" />
-            </geometry>
-        </collision>
-        <contact_coefficients mu="200.0" kp="0.0" kd="0.0"/>
+            <origin xyz="${link6_len+left_gripper_len/2} -0.03 0"/>
+            <geometry>
+                <box size="${left_gripper_len} ${left_gripper_width} ${left_gripper_height}" />
+            </geometry>
+        </collision>
+        <contact_coefficients mu="1.0" kp="1.0" kd="1.0"/>
         <xacro:inertial_matrix mass="1"/>
     </link>
@@ -279,5 +279,5 @@
     <link name="gripper_finger_link2">
         <visual>
-            <origin xyz="0.04 0.03 0"/>
+            <origin xyz="${link6_len+right_gripper_len/2} 0.03 0.0"/>
             <geometry>
                 <box size="${right_gripper_len} ${right_gripper_width} ${right_gripper_height}" />
@@ -286,19 +286,19 @@
         </visual>
         <collision>
-            <origin xyz="0.04 0.03 0"/>
-            <geometry>
-                <box size="${right_gripper_len/2} ${right_gripper_width} ${right_gripper_height}" />
-            </geometry>
-        </collision>
-        <contact_coefficients mu="200.0" kp="0.0" kd="0.0"/>
+            <origin xyz="${link6_len+right_gripper_len/2} 0.03 0"/>
+            <geometry>
+                <box size="${right_gripper_len} ${right_gripper_width} ${right_gripper_height}" />
+            </geometry>
+        </collision>
+        <!-- <contact_coefficients mu="1.0" kp="1.0" kd="1.0"/> -->
         <xacro:inertial_matrix mass="1"/>
     </link>
     <!-- Grasping frame -->
-    <link name="grasping_frame"/>
+    <!-- <link name="grasping_frame"/>
     <joint name="grasping_frame_joint" type="fixed">
         <parent link="link6"/>
         <child link="grasping_frame"/>
         <origin xyz="0.08 0 0" rpy="0 0 0"/>
-    </joint>
+    </joint> -->
     <!-- /////////////////////////////////   camera   ////////////////////////////////////// -->
     <xacro:include filename="camera.xacro" />
@@ -361,17 +361,20 @@
             <robotNamespace>/arm</robotNamespace>
         </plugin>
+    </gazebo>
+    <gazebo>
         <plugin name="gazebo_grasp_fix" filename="libgazebo_grasp_fix.so">
             <arm>
                 <arm_name>arm</arm_name>
-                <!-- <palm_link> hand_link_name  </palm_link> -->
+                <palm_link> link6  </palm_link>
                 <gripper_link> gripper_finger_link1 </gripper_link>
+                <palm_link> link6  </palm_link>
                 <gripper_link> gripper_finger_link2 </gripper_link>
             </arm>
-            <forces_angle_tolerance>100</forces_angle_tolerance>
-            <update_rate>4</update_rate>
-            <grip_count_threshold>4</grip_count_threshold>
+            <forces_angle_tolerance>150</forces_angle_tolerance>
+            <update_rate>130</update_rate>
+            <grip_count_threshold>1</grip_count_threshold>
             <max_grip_count>8</max_grip_count>
-            <release_tolerance>0.005</release_tolerance>
-            <disable_collisions_on_attach>false</disable_collisions_on_attach>
+            <release_tolerance>0.1</release_tolerance>
+            <disable_collisions_on_attach>true</disable_collisions_on_attach>
             <contact_topic>__default_topic__</contact_topic>
         </plugin>

Commit message: arm consistence

File: ros_arm/arm/xacro/arm.xacro (robot description, xacro)
@@ -282,13 +282,7 @@
     <link name="grasping_frame"/>
     <joint name="grasping_frame_joint" type="fixed">
-<<<<<<< Updated upstream
-      <parent link="link6"/>
-      <child link="grasping_frame"/>
-      <origin xyz="0.08 0 0" rpy="0 0 0"/>
-=======
         <parent link="link6"/>
         <child link="grasping_frame"/>
         <origin xyz="0.08 0 0" rpy="0 0 .02"/>
->>>>>>> Stashed changes
     </joint>
     <!-- /////////////////////////////////   camera   ////////////////////////////////////// -->
@@ -380,6 +374,4 @@
             <robotNamespace>/arm</robotNamespace>
         </plugin>
-<<<<<<< Updated upstream
-=======
         <plugin name="gazebo_grasp_fix" filename="libgazebo_grasp_fix.so">
             <arm>
@@ -397,5 +389,4 @@
             <contact_topic>__default_topic__</contact_topic>
         </plugin>
->>>>>>> Stashed changes
     </gazebo>
 </robot>

Commit message: arm

File: ros_arm/arm/xacro/arm.xacro (robot description, xacro)
@@ -299,9 +299,5 @@
         <parent link="link6"/>
         <child link="grasping_frame"/>
-<<<<<<< HEAD
-        <origin xyz="0.08 0 0" rpy="0 0 .02"/>
-=======
         <origin xyz="0.08 0 0" rpy="0 0 0"/>
->>>>>>> origin/master
     </joint>
     <!-- /////////////////////////////////   camera   ////////////////////////////////////// -->
@@ -396,11 +392,4 @@
             <arm>
                 <arm_name>arm</arm_name>
-<<<<<<< HEAD
-                <palm_link> link6 </palm_link>
-                <gripper_link> gripper_finger_link1 </gripper_link>
-                <gripper_link> gripper_finger_link2 </gripper_link>
-            </arm>
-            <forces_angle_tolerance>120</forces_angle_tolerance>
-=======
                 <!-- <palm_link> hand_link_name  </palm_link> -->
                 <gripper_link> gripper_finger_link1 </gripper_link>
@@ -408,5 +397,4 @@
             </arm>
             <forces_angle_tolerance>100</forces_angle_tolerance>
->>>>>>> origin/master
             <update_rate>4</update_rate>
             <grip_count_threshold>4</grip_count_threshold>
