Commit message: add a1 and own dog in ros_dog/dog

File: ros_dog/dog/xacro/dog.xacro (robot description, xacro)
@@ -45,5 +45,5 @@
     </xacro:macro>
     <!-- base_link -->
-    <link name="base_link">
+    <!-- <link name="base_link">
         <visual>
             <origin xyz="0 0 ${body_h}" rpy="0 0 0" />
@@ -59,5 +59,5 @@
             </geometry>
         </collision>
-    </link>
+    </link> -->
     <!-- body_link -->
     <link name="body_link">
@@ -75,5 +75,5 @@
             </geometry>
         </collision>
-        <xacro:inertial_matrix mass="1.0" />
+        <xacro:inertial_matrix mass="10.0" />
     </link>
     <!-- leg -->
@@ -93,5 +93,5 @@
                 </geometry>
             </collision>
-            <xacro:inertial_matrix mass="1.0" />
+            <xacro:inertial_matrix mass="10.0" />
         </link>
         <link name="${leg_name}_thigh_link">
@@ -109,5 +109,5 @@
                 </geometry>
             </collision>
-            <xacro:inertial_matrix mass="1.0" />
+            <xacro:inertial_matrix mass="10.0" />
         </link>
         <link name="${leg_name}_feet_link">
@@ -125,5 +125,5 @@
                 </geometry>
             </collision>
-            <xacro:inertial_matrix mass="1.0" />
+            <xacro:inertial_matrix mass="10.0" />
         </link>
         <joint name="${leg_name}_keen_joint" type="revolute">
@@ -132,6 +132,6 @@
             <child link="${leg_name}_thigh_link" />
             <axis xyz="0 0 1" />
-            <limit effort="300.0" lower="-${M_PI/2}" upper="${M_PI/2}" velocity="1" />
-            <dynamics damping="50" friction="1" />
+            <limit effort="300.0" lower="-${M_PI}" upper="${M_PI}" velocity="1" />
+            <dynamics damping="0" friction="0.5" />
         </joint>
         <joint name="${leg_name}_feet_joint" type="fixed">
@@ -149,10 +149,10 @@
     <xacro:leg leg_name="right_forward_leg" />
     <xacro:leg leg_name="right_back_leg" />
-    <!-- base_body_joint -->
+    <!-- base_body_joint
     <joint name="base_body_joint" type="fixed">
         <origin xyz="0 0 ${body_h}" rpy="3.14 0 0" />
         <parent link="base_link" />
         <child link="body_link" />
-    </joint>
+    </joint> -->
     <!-- leg_body_joint -->
     <joint name="left_forward_leg_body_joint" type="revolute">
@@ -162,5 +162,5 @@
         <axis xyz="0 0 1" />
         <limit effort="300" lower="-${M_PI/2}" upper="${M_PI/2}" velocity="1" />
-        <dynamics damping="50" friction="1" />
+        <dynamics damping="0" friction="0.5" />
     </joint>
     <joint name="left_back_leg_body_joint" type="revolute">
@@ -170,5 +170,5 @@
         <axis xyz="0 0 1" />
         <limit effort="300" lower="-${M_PI/2}" upper="${M_PI/2}" velocity="1" />
-        <dynamics damping="50" friction="1" />
+        <dynamics damping="0" friction="0.5" />
     </joint>
     <joint name="right_forward_leg_body_joint" type="revolute">
@@ -178,13 +178,19 @@
         <axis xyz="0 0 1" />
         <limit effort="300" lower="-${M_PI/2}" upper="${M_PI/2}" velocity="1" />
-        <dynamics damping="50" friction="1" />
+        <dynamics damping="0" friction="0.5" />
     </joint>
     <joint name="right_back_leg_body_joint" type="revolute">
-        <origin xyz="-${body_link_length/2} -${body_link_width/2+calf_height/2} 0" rpy="1.57 0.785 0" />
+        <origin xyz="-${body_link_length/2} -${body_link_width/2+calf_height/2} 0" rpy="1.57 0 0" />
         <parent link="body_link" />
         <child link="right_back_leg_calf_link" />
         <axis xyz="0 0 1" />
         <limit effort="300" lower="-${M_PI/2}" upper="${M_PI/2}" velocity="0.00005" />
-        <dynamics damping="50" friction="1" />
+        <dynamics damping="0" friction="0.5" />
     </joint>
+    <!-- ros_control plugin -->
+    <gazebo>
+        <plugin name="gazebo_ros_control" filename="libgazebo_ros_control.so">
+            <robotNamespace>/arm</robotNamespace>
+        </plugin>
+    </gazebo>
 </robot>

Commit message: 1. fixed wrongs in dog.xacro 2. add an example of pig_dog: dog2.xacro

File: ros_dog/dog/xacro/dog.xacro (robot description, xacro)
@@ -41,13 +41,29 @@
         <inertial>
             <mass value="${mass}" />
-            <inertia ixx="1.0" ixy="0.0" ixz="0.0" iyy="1.0" iyz="0.0" izz="1.0" />
+            <inertia ixx="0.166667" ixy="0" ixz="0" iyy="0.166667" iyz="0" izz="0.166667"/>
         </inertial>
     </xacro:macro>
     <!-- base_link -->
-    <!-- <link name="base_link">
+    <link name="base_link">
         <visual>
-            <origin xyz="0 0 ${body_h}" rpy="0 0 0" />
+            <origin xyz="0 0 0" rpy="0 0 0" />
             <geometry>
                 <box size="${body_link_length/10} ${body_link_width/10} ${body_link_height/10}" />
+            </geometry>
+            <material name="White" />
+        </visual>
+        <!-- <collision>
+            <origin xyz="0 0 0" rpy="0 0 0" />
+            <geometry>
+                <box size="${body_link_length/10} ${body_link_width/10} ${body_link_height/10}" />
+            </geometry>
+        </collision> -->
+    </link>
+    <!-- body_link -->
+    <link name="body_link">
+        <visual>
+            <origin xyz="0 0 0" rpy="0 0 0" />
+            <geometry>
+                <box size="${body_link_length} ${body_link_width} ${body_link_height}" />
             </geometry>
             <material name="White" />
@@ -56,24 +72,8 @@
             <origin xyz="0 0 0" rpy="0 0 0" />
             <geometry>
-                <box size="${body_link_length/10} ${body_link_width/10} ${body_link_height/10}" />
+                <box size="${body_link_length} ${body_link_width} ${body_link_height}" />
             </geometry>
         </collision>
-    </link> -->
-    <!-- body_link -->
-    <link name="body_link">
-        <visual>
-            <origin xyz="0 0 0" rpy="0 0 0" />
-            <geometry>
-                <box size="${body_link_length} ${body_link_width} ${body_link_height}" />
-            </geometry>
-            <material name="White" />
-        </visual>
-        <collision>
-            <origin xyz="0 0 0" rpy="0 0 0" />
-            <geometry>
-                <box size="${body_link_length} ${body_link_width} ${body_link_height}" />
-            </geometry>
-        </collision>
-        <xacro:inertial_matrix mass="10.0" />
+        <xacro:inertial_matrix mass="5" />
     </link>
     <!-- leg -->
@@ -88,10 +88,10 @@
             </visual>
             <collision>
-                <origin xyz="0 0 0" rpy="0 0 0" />
+                <origin xyz="0 ${calf_len/2} 0" rpy="0 0 0" />
                 <geometry>
                     <box size="${calf_width} ${calf_len} ${calf_height}" />
                 </geometry>
             </collision>
-            <xacro:inertial_matrix mass="10.0" />
+            <xacro:inertial_matrix mass="0.5" />
         </link>
         <link name="${leg_name}_thigh_link">
@@ -104,10 +104,10 @@
             </visual>
             <collision>
-                <origin xyz="0 0 0" rpy="0 0 0" />
+                <origin xyz="0 ${thigh_len/2} 0" rpy="0 0 0" />
                 <geometry>
                     <box size="${thigh_width} ${thigh_len} ${thigh_height}" />
                 </geometry>
             </collision>
-            <xacro:inertial_matrix mass="10.0" />
+            <xacro:inertial_matrix mass="0.5" />
         </link>
         <link name="${leg_name}_feet_link">
@@ -120,10 +120,14 @@
             </visual>
             <collision>
-                <origin xyz="0 0 0" rpy="0 0 0" />
+                <origin xyz="0 ${thigh_len/2} 0" rpy="0 0 0" />
                 <geometry>
                     <sphere radius="${point_feet_radius}" />
                 </geometry>
             </collision>
-            <xacro:inertial_matrix mass="10.0" />
+            <inertial>
+                <mass value="0.1"/>
+                <origin rpy="0 0 0" xyz="0 0 0"/>
+                <inertia ixx="0.1" ixy="0" ixz="0" iyy="0.1" iyz="0" izz="0.1"/>
+            </inertial>
         </link>
         <joint name="${leg_name}_keen_joint" type="revolute">
@@ -133,5 +137,5 @@
             <axis xyz="0 0 1" />
             <limit effort="300.0" lower="-${M_PI}" upper="${M_PI}" velocity="1" />
-            <dynamics damping="0" friction="0.5" />
+            <dynamics damping="0" friction="0.1" />
         </joint>
         <joint name="${leg_name}_feet_joint" type="fixed">
@@ -140,6 +144,6 @@
             <child link="${leg_name}_feet_link" />
             <axis xyz="0 0 1" />
-            <limit effort="300.0" lower="-${M_PI/2}" upper="${M_PI/2}" velocity="1" />
-            <dynamics damping="50" friction="1" />
+            <!-- <limit effort="300.0" lower="-${M_PI/2}" upper="${M_PI/2}" velocity="1" /> -->
+            <!-- <dynamics damping="0" friction="0.1" /> -->
         </joint>
     </xacro:macro>
@@ -149,10 +153,10 @@
     <xacro:leg leg_name="right_forward_leg" />
     <xacro:leg leg_name="right_back_leg" />
-    <!-- base_body_joint
+    <!-- base_body_joint -->
     <joint name="base_body_joint" type="fixed">
-        <origin xyz="0 0 ${body_h}" rpy="3.14 0 0" />
+        <origin xyz="0 0 0" rpy="3.14 0 0" />
         <parent link="base_link" />
         <child link="body_link" />
-    </joint> -->
+    </joint>
     <!-- leg_body_joint -->
     <joint name="left_forward_leg_body_joint" type="revolute">
@@ -162,5 +166,5 @@
         <axis xyz="0 0 1" />
         <limit effort="300" lower="-${M_PI/2}" upper="${M_PI/2}" velocity="1" />
-        <dynamics damping="0" friction="0.5" />
+        <dynamics damping="0" friction="0.1" />
     </joint>
     <joint name="left_back_leg_body_joint" type="revolute">
@@ -170,5 +174,5 @@
         <axis xyz="0 0 1" />
         <limit effort="300" lower="-${M_PI/2}" upper="${M_PI/2}" velocity="1" />
-        <dynamics damping="0" friction="0.5" />
+        <dynamics damping="0" friction="0.1" />
     </joint>
     <joint name="right_forward_leg_body_joint" type="revolute">
@@ -178,13 +182,13 @@
         <axis xyz="0 0 1" />
         <limit effort="300" lower="-${M_PI/2}" upper="${M_PI/2}" velocity="1" />
-        <dynamics damping="0" friction="0.5" />
+        <dynamics damping="0" friction="0.1" />
     </joint>
     <joint name="right_back_leg_body_joint" type="revolute">
-        <origin xyz="-${body_link_length/2} -${body_link_width/2+calf_height/2} 0" rpy="1.57 0 0" />
+        <origin xyz="-${body_link_length/2} -${body_link_width/2+calf_height/2} 0" rpy="1.57 0.785 0" />
         <parent link="body_link" />
         <child link="right_back_leg_calf_link" />
         <axis xyz="0 0 1" />
-        <limit effort="300" lower="-${M_PI/2}" upper="${M_PI/2}" velocity="0.00005" />
-        <dynamics damping="0" friction="0.5" />
+        <limit effort="300" lower="-${M_PI/2}" upper="${M_PI/2}" velocity="1" />
+        <dynamics damping="0" friction="0.1" />
     </joint>
     <!-- ros_control plugin -->

Commit message: add controller in dog.xacro

File: ros_dog/dog/xacro/dog.xacro (robot description, xacro)
@@ -136,5 +136,5 @@
             <child link="${leg_name}_thigh_link" />
             <axis xyz="0 0 1" />
-            <limit effort="300.0" lower="-${M_PI}" upper="${M_PI}" velocity="1" />
+            <limit effort="300.0" lower="-${M_PI/2}" upper="${M_PI/2}" velocity="1" />
             <dynamics damping="0" friction="0.1" />
         </joint>
@@ -195,6 +195,27 @@
     <gazebo>
         <plugin name="gazebo_ros_control" filename="libgazebo_ros_control.so">
-            <robotNamespace>/arm</robotNamespace>
+            <robotNamespace>/dog</robotNamespace>
         </plugin>
     </gazebo>
+    <!-- Transmissions for ROS Control -->
+    <xacro:macro name="transmission_block" params="joint_name">
+        <transmission name="tran1">
+            <type>transmission_interface/SimpleTransmission</type>
+            <joint name="${joint_name}">
+                <hardwareInterface>hardware_interface/PositionJointInterface</hardwareInterface>
+            </joint>
+            <actuator name="motor1">
+                <hardwareInterface>hardware_interface/PositionJointInterface</hardwareInterface>
+                <mechanicalReduction>1</mechanicalReduction>
+            </actuator>
+        </transmission>
+    </xacro:macro>
+    <xacro:transmission_block joint_name="left_forward_leg_body_joint"/>
+    <xacro:transmission_block joint_name="left_forward_leg_keen_joint"/>
+    <xacro:transmission_block joint_name="left_back_leg_body_joint"/>
+    <xacro:transmission_block joint_name="left_back_leg_keen_joint"/>
+    <xacro:transmission_block joint_name="right_forward_leg_body_joint"/>
+    <xacro:transmission_block joint_name="right_forward_leg_keen_joint"/>
+    <xacro:transmission_block joint_name="right_back_leg_body_joint"/>
+    <xacro:transmission_block joint_name="right_back_leg_keen_joint"/>
 </robot>

Commit message: v1

File: ros_dog/dog/xacro/dog.xacro (robot description, xacro)
@@ -155,5 +155,5 @@
     <!-- base_body_joint -->
     <joint name="base_body_joint" type="fixed">
-        <origin xyz="0 0 0" rpy="3.14 0 0" />
+        <origin xyz="0 0 0" rpy="0 0 0" /> <!--up and down: rpy="3.14 0 0"-->
         <parent link="base_link" />
         <child link="body_link" />
@@ -200,10 +200,10 @@
     <!-- Transmissions for ROS Control -->
     <xacro:macro name="transmission_block" params="joint_name">
-        <transmission name="tran1">
+        <transmission name="tran_${joint_name}">
             <type>transmission_interface/SimpleTransmission</type>
             <joint name="${joint_name}">
                 <hardwareInterface>hardware_interface/PositionJointInterface</hardwareInterface>
             </joint>
-            <actuator name="motor1">
+            <actuator name="motor_${joint_name}">
                 <hardwareInterface>hardware_interface/PositionJointInterface</hardwareInterface>
                 <mechanicalReduction>1</mechanicalReduction>

Commit message: fixed most of the bug TODO: response = sefl.arm_mover()

File: ros_dog/dog/xacro/dog.xacro (robot description, xacro)
@@ -136,5 +136,5 @@
             <child link="${leg_name}_thigh_link" />
             <axis xyz="0 0 1" />
-            <limit effort="300.0" lower="-${M_PI/2}" upper="${M_PI/2}" velocity="1" />
+            <limit effort="300.0" lower="-${M_PI/2}" upper="${M_PI/2}" velocity="10" />
             <dynamics damping="0" friction="0.1" />
         </joint>
@@ -144,5 +144,5 @@
             <child link="${leg_name}_feet_link" />
             <axis xyz="0 0 1" />
-            <!-- <limit effort="300.0" lower="-${M_PI/2}" upper="${M_PI/2}" velocity="1" /> -->
+            <!-- <limit effort="300.0" lower="-${M_PI/2}" upper="${M_PI/2}" velocity="10" /> -->
             <!-- <dynamics damping="0" friction="0.1" /> -->
         </joint>
@@ -155,5 +155,6 @@
     <!-- base_body_joint -->
     <joint name="base_body_joint" type="fixed">
-        <origin xyz="0 0 0" rpy="0 0 0" /> <!--up and down: rpy="3.14 0 0"-->
+        <origin xyz="0 0 0" rpy="0 0 0" />
+        <!--up: rpy="3.14 0 0" down: rpy="0 0 0"-->
         <parent link="base_link" />
         <child link="body_link" />
@@ -165,5 +166,5 @@
         <child link="left_forward_leg_calf_link" />
         <axis xyz="0 0 1" />
-        <limit effort="300" lower="-${M_PI/2}" upper="${M_PI/2}" velocity="1" />
+        <limit effort="300" lower="-${M_PI/2}" upper="${M_PI/2}" velocity="10" />
         <dynamics damping="0" friction="0.1" />
     </joint>
@@ -173,5 +174,5 @@
         <child link="left_back_leg_calf_link" />
         <axis xyz="0 0 1" />
-        <limit effort="300" lower="-${M_PI/2}" upper="${M_PI/2}" velocity="1" />
+        <limit effort="300" lower="-${M_PI/2}" upper="${M_PI/2}" velocity="10" />
         <dynamics damping="0" friction="0.1" />
     </joint>
@@ -181,5 +182,5 @@
         <child link="right_forward_leg_calf_link" />
         <axis xyz="0 0 1" />
-        <limit effort="300" lower="-${M_PI/2}" upper="${M_PI/2}" velocity="1" />
+        <limit effort="300" lower="-${M_PI/2}" upper="${M_PI/2}" velocity="10" />
         <dynamics damping="0" friction="0.1" />
     </joint>
@@ -189,5 +190,5 @@
         <child link="right_back_leg_calf_link" />
         <axis xyz="0 0 1" />
-        <limit effort="300" lower="-${M_PI/2}" upper="${M_PI/2}" velocity="1" />
+        <limit effort="300" lower="-${M_PI/2}" upper="${M_PI/2}" velocity="10" />
         <dynamics damping="0" friction="0.1" />
     </joint>
