Commit message: zcy_newest

File: ros_dog/arm_dog/xacro/arm.xacro (robot description, xacro)
@@ -1,54 +1,83 @@
 <?xml version="1.0"?>
-<robot name="arm" xmlns:xacro="http://ros.org/wiki/xacro">
-<!-- Constants -->
+<robot name="arm"
+    xmlns:xacro="http://ros.org/wiki/xacro">
+    <!-- Defining the colors used in this robot -->
+    <material name="Black">
+        <color rgba="0 0 0 1"/>
+    </material>
+    <material name="White">
+        <color rgba="1 1 1 1"/>
+    </material>
+    <material name="Blue">
+        <color rgba="0 0 1 1"/>
+    </material>
+    <material name="Red">
+        <color rgba="1 0 0 1"/>
+    </material>
+    <!-- Constants -->
     <xacro:property name="M_PI" value="3.14159"/>
+    <!-- link1 properties -->
+    <xacro:property name="link1_width" value="0.03" />
+    <xacro:property name="link1_len" value="0.15" />
+    <!-- link2 properties -->
+    <xacro:property name="link2_width" value="0.03" />
+    <xacro:property name="link2_len" value="0.2" />
+    <!-- link3 properties -->
+    <xacro:property name="link3_width" value="0.03" />
+    <xacro:property name="link3_len" value="0.2" />
+    <!-- link4 properties -->
+    <xacro:property name="link4_width" value="0.025" />
+    <xacro:property name="link4_len" value="0.03" />
+    <!-- link5 properties -->
+    <xacro:property name="link5_width" value="0.03" />
+    <xacro:property name="link5_len" value="0.06" />
+    <!-- link6 properties -->
+    <xacro:property name="link6_width" value="0.04" />
+    <xacro:property name="link6_len" value="0.02" />
+    <!-- Left gripper -->
+    <xacro:property name="left_gripper_len" value="0.06" />
+    <xacro:property name="left_gripper_width" value="0.01" />
+    <xacro:property name="left_gripper_height" value="0.01" />
+    <!-- Right gripper -->
+    <xacro:property name="right_gripper_len" value="0.06" />
+    <xacro:property name="right_gripper_width" value="0.01" />
+    <xacro:property name="right_gripper_height" value="0.01" />
+    <!-- Gripper frame -->
+    <xacro:property name="grasp_frame_radius" value="0.001" />
     <!-- Inertial matrix -->
     <xacro:macro name="inertial_matrix" params="mass">
         <inertial>
             <mass value="${mass}" />
-            <inertia ixx="0.166667" ixy="0" ixz="0" iyy="0.166667" iyz="0" izz="0.166667"/>
+            <inertia ixx="1.0" ixy="0.0" ixz="0.0" iyy="0.5" iyz="0.0" izz="1.0" />
         </inertial>
     </xacro:macro>
-    <!-- base_link properties -->
-    <xacro:property name="base_link_width" value="0.06" />
-    <xacro:property name="base_link_len" value="0.005" />
-    <!-- link1 properties -->
-    <xacro:property name="link1_width" value="0.03" />
-    <xacro:property name="link1_len" value="0.03" />
-    <!-- link2 properties -->
-    <xacro:property name="link2_width" value="0.02" />
-    <xacro:property name="link2_len" value="0.2" />
-    <!-- link3 properties -->
-    <xacro:property name="link3_width" value="0.02" />
-    <xacro:property name="link3_len" value="0.2" />
-    <!-- link4 properties -->
-    <xacro:property name="link4_width" value="0.015" />
-    <xacro:property name="link4_len" value="0.03" />
-    <!-- link5 properties -->
-    <xacro:property name="link5_width" value="0.02" />
-    <xacro:property name="link5_len" value="0.05" />
-    <!-- link6 properties -->
-    <xacro:property name="link6_width" value="0.025" />
-    <xacro:property name="link6_len" value="0.02" />
-    <!-- Left gripper -->
-    <xacro:property name="left_gripper_len" value="0.08" />
-    <xacro:property name="left_gripper_width" value="0.01" />
-    <xacro:property name="left_gripper_height" value="0.01" />
-    <!-- Right gripper -->
-    <xacro:property name="right_gripper_len" value="0.08" />
-    <xacro:property name="right_gripper_width" value="0.01" />
-    <xacro:property name="right_gripper_height" value="0.01" />
-    <!-- Gripper frame -->
-    <xacro:property name="grasp_frame_radius" value="0.001" />
-    <joint name="body_arm_joint" type="fixed">
-        <origin xyz="${body_link_length*0.3} 0 ${body_link_height/2+base_link_len/2}" rpy="0 0 0" />
-        <parent link="body_link"/>
-        <child link="base_link"/>
-    </joint>
+    <!-- ///////////////////////////////////////   bottom_joint   ////////////////////////////////////////// -->
+    <joint name="bottom_joint" type="fixed">
+        <origin xyz="0 0 -0.025" rpy="0 0 0" />
+        <parent link="base_link"/>
+        <child link="bottom_link"/>
+    </joint>
+    <link name="bottom_link">
+        <visual>
+            <origin xyz=" 0 0 0" rpy="0 0 0"/>
+            <geometry>
+                <box size="0.1 0.1 0.01" />
+            </geometry>
+            <material name="Blue" />
+        </visual>
+        <collision>
+            <origin xyz=" 0 0 0" rpy="0 0 0"/>
+            <geometry>
+                <box size="0.1 0.1 0.01" />
+            </geometry>
+        </collision>
+        <xacro:inertial_matrix mass="1000"/>
+    </link>
+    <!-- /////////////////////////////////////   BASE LINK    ////////////////////////////////////////////// -->
     <link name="base_link">
         <visual>
             <origin xyz="0 0 0" rpy="0 0 0" />
             <geometry>
-                <box size="${base_link_width} ${base_link_width} ${base_link_len}" />
+                <box size="0.1 0.1 0.04" />
             </geometry>
             <material name="White" />
@@ -57,18 +86,18 @@
             <origin xyz="0 0 0" rpy="0 0 0" />
             <geometry>
-                <box size="${base_link_width/10} ${base_link_width/10} ${base_link_len/10}" />
-            </geometry>
-        </collision>
-        <xacro:inertial_matrix mass="0.001"/>
-    </link>
-    <!-- link1 -->
+                <box size="0.1 0.1 0.04" />
+            </geometry>
+        </collision>
+        <xacro:inertial_matrix mass="1"/>
+    </link>
     <joint name="joint1" type="revolute">
         <parent link="base_link"/>
         <child link="link1"/>
-        <origin xyz="0 0 0.0005" rpy="0 ${M_PI/2} 0" />
-        <axis xyz="-1 0 0" />
+        <origin xyz="0 0 0.02" rpy="0 ${M_PI/2} 0" />
+        <axis xyz="1 0 0" />
         <limit effort="300" velocity="1" lower="-2.96" upper="2.96"/>
         <dynamics damping="50" friction="1"/>
     </joint>
+    <!-- /////////////////////////////////////   LINK1  ////////////////////////////////////////////// -->
     <link name="link1">
         <visual>
@@ -82,10 +111,9 @@
             <origin xyz="-${link1_len/2} 0 0" rpy="0 ${M_PI/2} 0" />
             <geometry>
-                <cylinder radius="${link1_width}" length="${link1_len}"/>
-            </geometry>
-        </collision>
-        <xacro:inertial_matrix mass="0.01"/>
-    </link>
-    <!-- link2 -->
+                <cylinder radius="${link1_width/10}" length="${link1_len/10}"/>
+            </geometry>
+        </collision>
+        <xacro:inertial_matrix mass="1"/>
+    </link>
     <joint name="joint2" type="revolute">
         <parent link="link1"/>
@@ -96,4 +124,5 @@
         <dynamics damping="50" friction="1"/>
     </joint>
+    <!-- ///////////////////////////////////////   LINK2  ////////////////////////////////////////////// -->
     <link name="link2">
         <visual>
@@ -107,10 +136,9 @@
             <origin xyz="0 0 ${link2_len/2}" rpy="0 0 0" />
             <geometry>
-                <cylinder radius="${link2_width}" length="${link2_len}"/>
-            </geometry>
-        </collision>
-        <xacro:inertial_matrix mass="0.01"/>
-    </link>
-    <!-- link3 -->
+                <cylinder radius="${link2_width/10}" length="${link2_len/10}"/>
+            </geometry>
+        </collision>
+        <xacro:inertial_matrix mass="1"/>
+    </link>
     <joint name="joint3" type="revolute">
         <parent link="link2"/>
@@ -121,4 +149,5 @@
         <dynamics damping="50" friction="1"/>
     </joint>
+    <!-- /////////////////////////////////   LINK3  ///////////////////////////////////////////////////// -->
     <link name="link3">
         <visual>
@@ -132,10 +161,9 @@
             <origin xyz="0 0 -${link3_len/2}" rpy="0 0 0" />
             <geometry>
-                <cylinder radius="${link3_width}" length="${link3_len}"/>
-            </geometry>
-        </collision>
-        <xacro:inertial_matrix mass="0.01"/>
-    </link>
-    <!-- link4 -->
+                <cylinder radius="${link3_width/10}" length="${link3_len/10}"/>
+            </geometry>
+        </collision>
+        <xacro:inertial_matrix mass="1"/>
+    </link>
     <joint name="joint4" type="revolute">
         <parent link="link3"/>
@@ -146,4 +174,5 @@
         <dynamics damping="50" friction="1"/>
     </joint>
+    <!-- ///////////////////////////////////   LINK4  //////////////////////////////////////////////// -->
     <link name="link4">
         <visual>
@@ -160,15 +189,15 @@
             </geometry>
         </collision>
-        <xacro:inertial_matrix mass="0.01"/>
-    </link>
-    <!-- link5 -->
+        <xacro:inertial_matrix mass="1"/>
+    </link>
     <joint name="joint5" type="revolute">
         <parent link="link4"/>
         <child link="link5"/>
         <origin xyz="${link4_len} 0.0 0.0" rpy="0 ${M_PI/2} 0" />
-        <axis xyz="1 0 0" />
+        <axis xyz="-1 0 0" />
         <limit effort="300" velocity="1" lower="-2.62" upper="2.62" />
         <dynamics damping="50" friction="1"/>
     </joint>
+    <!-- //////////////////////////////////   LINK5  ///////////////////////////////////////////////// -->
     <link name="link5">
         <visual>
@@ -185,7 +214,6 @@
             </geometry>
         </collision>
-        <xacro:inertial_matrix mass="0.01"/>
-    </link>
-    <!-- link6 -->
+        <xacro:inertial_matrix mass="1"/>
+    </link>
     <joint name="joint6" type="revolute">
         <parent link="link5"/>
@@ -196,4 +224,5 @@
         <dynamics damping="50" friction="1"/>
     </joint>
+    <!-- ////////////////////////////////   LINK6  ///////////////////////////////////////////////// -->
     <link name="link6">
         <visual>
@@ -210,7 +239,6 @@
             </geometry>
         </collision>
-        <xacro:inertial_matrix mass="0.01"/>
-    </link>
-    <!-- finger_1 -->
+        <xacro:inertial_matrix mass="1"/>
+    </link>
     <joint name="finger_joint1" type="prismatic">
         <parent link="link6"/>
@@ -221,7 +249,9 @@
         <dynamics damping="50" friction="1"/>
     </joint>
+    <!-- //////////////////////////////////////   gripper   ////////////////////////////////////////////// -->
+    <!-- LEFT GRIPPER AFT LINK -->
     <link name="gripper_finger_link1">
         <visual>
-            <origin xyz="0.04 -0.03 0"/>
+            <origin xyz="${link6_len+left_gripper_len/2} -0.03 0"/>
             <geometry>
                 <box size="${left_gripper_len} ${left_gripper_width} ${left_gripper_height}" />
@@ -229,7 +259,13 @@
             <material name="White" />
         </visual>
-        <xacro:inertial_matrix mass="0.001"/>
-    </link>
-    <!-- finger_2 -->
+        <collision>
+            <origin xyz="${link6_len+left_gripper_len/2} -0.03 0"/>
+            <geometry>
+                <box size="${left_gripper_len} ${left_gripper_width} ${left_gripper_height}" />
+            </geometry>
+        </collision>
+        <contact_coefficients mu="1.0" kp="1.0" kd="1.0"/>
+        <xacro:inertial_matrix mass="1"/>
+    </link>
     <joint name="finger_joint2" type="prismatic">
         <parent link="link6"/>
@@ -240,7 +276,8 @@
         <dynamics damping="50" friction="1"/>
     </joint>
+    <!-- RIGHT GRIPPER AFT LINK -->
     <link name="gripper_finger_link2">
         <visual>
-            <origin xyz="0.04 0.03 0"/>
+            <origin xyz="${link6_len+right_gripper_len/2} 0.03 0.0"/>
             <geometry>
                 <box size="${right_gripper_len} ${right_gripper_width} ${right_gripper_height}" />
@@ -248,24 +285,62 @@
             <material name="White" />
         </visual>
-        <xacro:inertial_matrix mass="0.001"/>
+        <collision>
+            <origin xyz="${link6_len+right_gripper_len/2} 0.03 0"/>
+            <geometry>
+                <box size="${right_gripper_len} ${right_gripper_width} ${right_gripper_height}" />
+            </geometry>
+        </collision>
+        <!-- <contact_coefficients mu="1.0" kp="1.0" kd="1.0"/> -->
+        <xacro:inertial_matrix mass="1"/>
     </link>
     <!-- Grasping frame -->
-    <link name="grasping_frame"/>
+    <!-- <link name="grasping_frame"/>
     <joint name="grasping_frame_joint" type="fixed">
         <parent link="link6"/>
         <child link="grasping_frame"/>
         <origin xyz="0.08 0 0" rpy="0 0 0"/>
-    </joint>
+    </joint> -->
     <!-- /////////////////////////////////   camera   ////////////////////////////////////// -->
     <xacro:include filename="camera.xacro" />
     <xacro:include filename="camera_sensor.xacro" />
+    <!-- /////////////////////////////////   Gazebo   ////////////////////////////////////// -->
+    <gazebo reference="bottom_link">
+        <material>Gazebo/Black</material>
+    </gazebo>
+    <gazebo reference="base_link">
+        <material>Gazebo/White</material>
+    </gazebo>
+    <gazebo reference="link1">
+        <material>Gazebo/Blue</material>
+    </gazebo>
+    <gazebo reference="link2">
+        <material>Gazebo/White</material>
+    </gazebo>
+    <gazebo reference="link3">
+        <material>Gazebo/Blue</material>
+    </gazebo>
+    <gazebo reference="link4">
+        <material>Gazebo/Black</material>
+    </gazebo>
+    <gazebo reference="link5">
+        <material>Gazebo/White</material>
+    </gazebo>
+    <gazebo reference="link6">
+        <material>Gazebo/Blue</material>
+    </gazebo>
+    <gazebo reference="gripper_finger_link1">
+        <material>Gazebo/White</material>
+    </gazebo>
+    <gazebo reference="gripper_finger_link2">
+        <material>Gazebo/White</material>
+    </gazebo>
     <!-- Transmissions for ROS Control -->
     <xacro:macro name="transmission_block" params="joint_name">
-        <transmission name="tran_arm">
+        <transmission name="tran1">
             <type>transmission_interface/SimpleTransmission</type>
             <joint name="${joint_name}">
                 <hardwareInterface>hardware_interface/PositionJointInterface</hardwareInterface>
             </joint>
-            <actuator name="motor_arm">
+            <actuator name="motor1">
                 <hardwareInterface>hardware_interface/PositionJointInterface</hardwareInterface>
                 <mechanicalReduction>1</mechanicalReduction>
@@ -287,3 +362,21 @@
         </plugin>
     </gazebo>
+    <gazebo>
+        <plugin name="gazebo_grasp_fix" filename="libgazebo_grasp_fix.so">
+            <arm>
+                <arm_name>arm</arm_name>
+                <palm_link> link6  </palm_link>
+                <gripper_link> gripper_finger_link1 </gripper_link>
+                <palm_link> link6  </palm_link>
+                <gripper_link> gripper_finger_link2 </gripper_link>
+            </arm>
+            <forces_angle_tolerance>150</forces_angle_tolerance>
+            <update_rate>130</update_rate>
+            <grip_count_threshold>1</grip_count_threshold>
+            <max_grip_count>8</max_grip_count>
+            <release_tolerance>0.001</release_tolerance>
+            <disable_collisions_on_attach>true</disable_collisions_on_attach>
+            <contact_topic>__default_topic__</contact_topic>
+        </plugin>
+    </gazebo>
 </robot>
